Commit message: Added most things for the simulator

File: src/robot_description/igvc.urdf (robot description, URDF)
Before this commit: robot visual, 7 links, 6 joints
Links:
- link hokuyo_link: geometry collision box size=0.1 0.1 0.1; visual mesh filename=file:///home/blanknc/igvc_ws/src/robot_description/meshes/h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
Joints:
- joint hokuyo_joint: origin xyz=0 0 0 rpy=0 0 0 -> xyz=.6 0 0 rpy=0 0 0
