Commit message: Added a bunch of stuff, hope it works

File: src/robot_description/urdf/igvc.xacro (robot description, xacro)
@@ -244,5 +244,5 @@
       <origin xyz="0 0 0" rpy="0 0 0"/>
       <geometry>
-        <mesh filename="file:///home/blanknc/igvc_ws/src/robot_description/meshes/hokuyo.dae"/>
+        <mesh filename="package://robot_description/meshes/hokuyo.dae"/>
       </geometry>
     </visual>
@@ -258,12 +258,13 @@
   <xacro:robot_wheel fb="back" lr="right" parent="base_link" sideX="0.33" sideY="-0.325" sideZ="-.24" />
   <xacro:robot_wheel fb="front" lr="right" parent="base_link" sideX="-0.33" sideY="-0.325" sideZ="-.24" />
+<!--
 <gazebo>
       <plugin name="object_controller" filename="libgazebo_ros_planar_move.so">
         <commandTopic>cmd_vel</commandTopic>
-        <odometryTopic>odom</odometryTopic>
-        <odometryFrame>odom</odometryFrame>
+        <odometryTopic>odom2</odometryTopic>
+        <odometryFrame>odom2</odometryFrame>
         <odometryRate>20.0</odometryRate>
         <robotBaseFrame>base_link</robotBaseFrame>
       </plugin>
-    </gazebo>
+    </gazebo> -->
 </robot>
